File: remote control iot.kicad_sch (KiCad schematic)
At the start: 13 parts, among them K1 Fujitsu_FTR-LYAA005x, Q1 BC547, SW2 SW_Push, U1 Olimex_MOD-WIFI-ESP8266-DEV, U2 AMS1117-3.3

Commit message: Add files via upload
Parts:
- U1: footprint Module:Olimex_MOD-WIFI-ESP8266-DEV -> Module:Adafruit_HUZZAH_ESP8266_breakout_WithMountingHoles
Changed lines of the file:
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@@
 			)
 		)
-		(property "Footprint" "Module:Olimex_MOD-WIFI-ESP8266-DEV"
+		(property "Footprint" "Module:Adafruit_HUZZAH_ESP8266_breakout_WithMountingHoles"
 			(at 120.65 119.38 0)
 			(effects
